File: design_files/ASD2116.brd (EAGLE design)
At the start: 20 x 20 mm, 11 parts, among them J1 DF12-32-DP, J2 DF12-32-DS, U1 SPBTLE-RF, U2 TXB0104, U3 XC6217A33

Commit message: update format
Parts:
- removed C12, C4: 10uF, tinycircuits:C0603
- removed R6: 100K, tinycircuits:0402
- removed U3: XC6217A33, tinycircuits:SOT-25
- added C1, C2: 10uF, tinycircuits:C0603
- added R1: 100K, tinycircuits:0402
- added U4: BMD-100, tinycircuits:BMD-100
- U1: value SPBTLE-RF -> XC6217A33; device tinycircuits:SPBTLE-RF -> tinycircuits:SOT-25
- moved U1 7.57 mm to (27.6, 23.6), turned to 90 degrees
- moved U2 0.50 mm to (27.7, 17.4)
Connections:
- net CS_3V3: now also U4.14; no longer U1.10
- net GND: now also C1.2, C2.2, U1.2, U1.4, U4.1, U4.11, U4.2, U4.20, U4.3, U4.7, U4.9, U4.A, U4.B, U4.C, U4.D, U4.E, U4.F; no longer C12.2, C4.2, U1.6, U3.2, U3.4
- net IRQ: now also U4.18; no longer U1.4
- net MISO: now also U4.15; no longer U1.8
- net MOSI_3V3: now also U4.16; no longer U1.9
- net RESET_3V3: now also R1.2, U4.13; no longer R6.2, U1.11
- net SCK_3V3: now also U4.17; no longer U1.7
- net VCC: now also C1.1, U1.1, U1.3; no longer C4.1, U3.1, U3.3
- net VCC_3V3: now also C2.1, R1.1, U4.19; no longer C12.1, R6.1, U3.5
Routing:
- net VCC_3V3: track 33.2 -> 13.8 mm, vias 2 -> 0
- net VCC: track 36.2 -> 24.7 mm, vias 3 -> 1
- net MISO: track 14.6 -> 8.17 mm
- net SCK_3V3: track 1.78 -> 7.99 mm, vias 0 -> 2
- net RESET_3V3: track 8.55 -> 14.5 mm, vias 0 -> 2
- net CS_3V3: track 6.49 -> 11.5 mm, vias 0 -> 2
- net IRQ: track 11.3 -> 14.3 mm
- net MOSI_3V3: track 5.02 -> 6.86 mm
- net SS: track 20.0 -> 19.5 mm
- net SCK: track 12.5 -> 12.0 mm
- net MOSI: track 17.6 -> 17.1 mm
- net IO9: track 19.3 -> 18.8 mm
- net GND: vias 31 -> 40
Other:
- board size 20 x 20 mm -> 22.5 x 21.3 mm
- board text added: "2"
- board text added: "ASD2116 - Rev2"
- board text added: "^ V-SCORE EDGE ALONG OUTLINE ^"
- board text removed: "1"
- board text removed: "ASD2116 - Rev1"
