File: design_files/ASD2116.sch (EAGLE design)
At the start: 10 parts, among them J1 DF12-32-DP, J2 DF12-32-DS, U1 SPBTLE-RF, U2 TXB0104, U3 XC6217A33

Commit message: update format
Parts:
- removed U3: XC6217A33, tinycircuits:AS-ITM-00249
- added U4: BMD-100, tinycircuits:AS-ITM-00402
- U1: value SPBTLE-RF -> XC6217A33; device tinycircuits:AS-ITM-00294 -> tinycircuits:AS-ITM-00249; PARTNO (none) -> AS-ITM-00249; VALUE (none) -> XC6217A33
- renumbered C12 to C2, C4 to C1, R6 to R1
Connections:
- net CS_3V3: now also U4.CS; no longer U1.CS
- net GND: now also U1.NC/GO, U1.VSS, U4.GND; no longer U1.GND, U3.NC/GO, U3.VSS
- net IRQ: now also U4.IRQ; no longer U1.IRQ
- net MISO: now also U4.MISO; no longer U1.MISO
- net MOSI_3V3: now also U4.MOSI; no longer U1.MOSI
- net RESET_3V3: now also U4.RESET; no longer U1.RESET
- net SCK_3V3: now also U4.SCLK; no longer U1.SCLK
- net VCC: now also U1.CE, U1.VIN; no longer U3.CE, U3.VIN
- net VCC_3V3: now also U1.VOUT, U4.VIN; no longer U1.VIN, U3.VOUT
Other:
- note added: "2"
- note added: "Hand Populated: -"
- note added: "Hand Soldered: -"
- note added: "Non Populated: -"
- note added: "Notes: -"
- note added: "Variant: Standard"
- note removed: "1"
Changed lines of the file:
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@@
 <part name="U2" library="tinycircuits" deviceset="AS-ITM-00048" device="" value="TXB0104"/>
 <part name="VCC5" library="tinycircuits" deviceset="VCC" device="" value="VCC"/>
-<part name="U3" library="tinycircuits" deviceset="AS-ITM-00249" device="" value="XC6217A33">
+<part name="U1" library="tinycircuits" deviceset="AS-ITM-00249" device="" value="XC6217A33">
 <attribute name="PARTNO" value="AS-ITM-00249"/>
 <attribute name="VALUE" value="XC6217A33"/>
@@
 <part name="GND9" library="tinycircuits" deviceset="GND" device=""/>
 <part name="GND10" library="tinycircuits" deviceset="GND" device=""/>
-<part name="C4" library="tinycircuits" deviceset="AS-ITM-00002" device="" value="10uF">
+<part name="C1" library="tinycircuits" deviceset="AS-ITM-00002" device="" value="10uF">
 <attribute name="PARTNO" value="AS-ITM-00002"/>
 </part>
-<part name="C12" library="tinycircuits" deviceset="AS-ITM-00002" device="" value="10uF">
+<part name="C2" library="tinycircuits" deviceset="AS-ITM-00002" device="" value="10uF">
 <attribute name="PARTNO" value="AS-ITM-00002"/>
 <attribute name="VALUE" value="10uF"/>
@@
 <attribute name="VALUE" value="0.0"/>
 </part>
-<part name="R6" library="tinycircuits" deviceset="AS-ITM-00004" device="" value="100K"/>
+<part name="R1" library="tinycircuits" deviceset="AS-ITM-00004" device="" value="100K"/>
 <part name="GND6" library="tinycircuits" deviceset="GND" device=""/>
-<part name="U1" library="tinycircuits" deviceset="AS-ITM-00294" device="" value="SPBTLE-RF"/>
 <part name="GND4" library="tinycircuits" deviceset="GND" device=""/>
+<part name="U4" library="tinycircuits" deviceset="AS-ITM-00402" device="" value="BMD-100"/>
 </parts>
 <sheets>
@@
 <text x="340.868" y="17.272" size="3.556" layer="94" font="vector">TinyShield - ST BLE</text>
 <text x="327.152" y="6.35" size="3.556" layer="94" font="vector">AS-SCH-ASD2116</text>
-<text x="416.56" y="6.858" size="3.556" layer="94" font="vector">1</text>
+<text x="416.56" y="6.858" size="3.556" layer="94" font="vector">2</text>
 <text x="299.72" y="142.24" size="3.81" layer="94" font="vector">TinyShield Expansion - Top</text>
 <text x="353.06" y="124.714" size="1.778" layer="91">IOREF</text>
@@
 <text x="203.962" y="117.094" size="2.54" layer="94" font="vector">R2 populated by defualt</text>
 <text x="203.962" y="112.014" size="2.54" layer="94" font="vector">R3 non-populated by default</text>
+<text x="48.26" y="63.5" size="1.778" layer="96">Variant: Standard</text>
+<text x="48.26" y="60.96" size="1.778" layer="96">Non Populated: -</text>
+<text x="48.26" y="58.42" size="1.778" layer="96">Hand Populated: -</text>
+<text x="48.26" y="55.88" size="1.778" layer="96">Hand Soldered: -</text>
+<text x="48.26" y="53.34" size="1.778" layer="96">Notes: -</text>
 </plain>
 <instances>
@@
 <attribute name="VALUE" x="195.58" y="220.98" size="1.778" layer="96" rot="R180"/>
 </instance>
-<instance part="U3" gate="G$1" x="99.06" y="210.82"/>
+<instance part="U1" gate="G$1" x="99.06" y="210.82"/>
 <instance part="GND2" gate="1" x="193.04" y="193.04"/>
 <instance part="GND3" gate="1" x="68.58" y="198.12"/>
@@
 <instance part="GND9" gate="1" x="370.84" y="190.5"/>
 <instance part="GND10" gate="1" x="370.84" y="104.14"/>
-<instance part="C4" gate="G$1" x="68.58" y="208.28"/>
-<instance part="C12" gate="G$1" x="129.54" y="208.28"/>
+<instance part="C1" gate="G$1" x="68.58" y="208.28"/>
+<instance part="C2" gate="G$1" x="129.54" y="208.28"/>
 <instance part="GND1" gate="1" x="129.54" y="198.12"/>
 <instance part="R2" gate="G$1" x="177.8" y="119.38"/>
 <instance part="R3" gate="G$1" x="177.8" y="111.76"/>
-<instance part="R6" gate="G$1" x="91.44" y="114.3"/>
+<instance part="R1" gate="G$1" x="91.44" y="114.3"/>
 <instance part="GND6" gate="1" x="106.68" y="96.52"/>
-<instance part="U1" gate="G$1" x="129.54" y="116.84"/>
 <instance part="GND4" gate="1" x="116.84" y="198.12"/>
+<instance part="U4" gate="G$1" x="129.54" y="116.84"/>
 </instances>
 <busses>
@@
 <wire x1="144.78" y1="119.38" x2="154.94" y2="119.38" width="0.1524" layer="91"/>
 <label x="149.86" y="119.38" size="1.778" layer="95"/>
-<pinref part="U1" gate="G$1" pin="MISO"/>
+<pinref part="U4" gate="G$1" pin="MISO"/>
 </segment>
 </net>
@@
 <junction x="68.58" y="213.36"/>
 <junction x="81.28" y="213.36"/>
-<pinref part="U3" gate="G$1" pin="CE"/>
-<pinref part="U3" gate="G$1" pin="VIN"/>
-<pinref part="C4" gate="G$1" pin="1"/>
+<pinref part="U1" gate="G$1" pin="CE"/>
+<pinref part="U1" gate="G$1" pin="VIN"/>
+<pinref part="C1" gate="G$1" pin="1"/>
 </segment>
 <segment>
@@
 <wire x1="144.78" y1="213.36" x2="129.54" y2="213.36" width="0.1524" layer="91"/>
 <label x="133.223" y="213.9188" size="1.778" layer="95"/>
-<pinref part="U3" gate="G$1" pin="VOUT"/>
-<pinref part="C12" gate="G$1" pin="1"/>
+<pinref part="U1" gate="G$1" pin="VOUT"/>
+<pinref part="C2" gate="G$1" pin="1"/>
 <wire x1="129.54" y1="213.36" x2="111.76" y2="213.36" width="0.1524" layer="91"/>
 <wire x1="129.54" y1="210.82" x2="129.54" y2="213.36" width="0.1524" layer="91"/>
@@
 <segment>
 <wire x1="114.3" y1="124.46" x2="83.82" y2="124.46" width="0.1524" layer="91"/>
-<pinref part="R6" gate="G$1" pin="1"/>
+<pinref part="R1" gate="G$1" pin="1"/>
 <wire x1="86.36" y1="114.3" x2="83.82" y2="114.3" width="0.1524" layer="91"/>
 <wire x1="83.82" y1="114.3" x2="83.82" y2="124.46" width="0.1524" layer="91"/>
@@
 <wire x1="83.82" y1="124.46" x2="71.12" y2="124.46" width="0.1524" layer="91"/>
 <label x="71.12" y="124.46" size="1.778" layer="95"/>
-<pinref part="U1" gate="G$1" pin="VIN"/>
+<pinref part="U4" gate="G$1" pin="VIN"/>
 </segment>
 </net>
@@
 <segment>
 <pinref part="GND3" gate="1" pin="GND"/>
-<pinref part="C4" gate="G$1" pin="2"/>
+<pinref part="C1" gate="G$1" pin="2"/>
 <wire x1="68.58" y1="200.66" x2="68.58" y2="203.2" width="0.1524" layer="91"/>
 </segment>
@@
 <wire x1="83.82" y1="208.28" x2="81.28" y2="208.28" width="0.1524" layer="91"/>
 <wire x1="81.28" y1="208.28" x2="81.28" y2="200.66" width="0.1524" layer="91"/>
-<pinref part="U3" gate="G$1" pin="VSS"/>
+<pinref part="U1" gate="G$1" pin="VSS"/>
 <pinref part="GND5" gate="1" pin="GND"/>
 </segment>
@@
 <segment>
 <pinref part="GND1" gate="1" pin="GND"/>
-<pinref part="C12" gate="G$1" pin="2"/>
+<pinref part="C2" gate="G$1" pin="2"/>
 <wire x1="129.54" y1="200.66" x2="129.54" y2="203.2" width="0.1524" layer="91"/>
 </segment>
@@
 <wire x1="106.68" y1="109.22" x2="106.68" y2="99.06" width="0.1524" layer="91"/>
 <pinref part="GND6" gate="1" pin="GND"/>
-<pinref part="U1" gate="G$1" pin="GND"/>
-</segment>
-<segment>
-<pinref part="U3" gate="G$1" pin="NC/GO"/>
+<pinref part="U4" gate="G$1" pin="GND"/>
+</segment>
+<segment>
+<pinref part="U1" gate="G$1" pin="NC/GO"/>
 <wire x1="111.76" y1="208.28" x2="116.84" y2="208.28" width="0.1524" layer="91"/>
 <wire x1="116.84" y1="208.28" x2="116.84" y2="200.66" width="0.1524" layer="91"/>
@@
 <wire x1="144.78" y1="116.84" x2="154.94" y2="116.84" width="0.1524" layer="91"/>
 <label x="149.86" y="116.84" size="1.778" layer="95"/>
-<pinref part="U1" gate="G$1" pin="SCLK"/>
+<pinref part="U4" gate="G$1" pin="SCLK"/>
 </segment>
 <segment>
@@
 <wire x1="144.78" y1="121.92" x2="154.94" y2="121.92" width="0.1524" layer="91"/>
 <label x="149.86" y="121.92" size="1.778" layer="95"/>
-<pinref part="U1" gate="G$1" pin="MOSI"/>
+<pinref part="U4" gate="G$1" pin="MOSI"/>
 </segment>
 <segment>
@@
 <wire x1="144.78" y1="124.46" x2="154.94" y2="124.46" width="0.1524" layer="91"/>
 <label x="149.86" y="124.46" size="1.778" layer="95"/>
-<pinref part="U1" gate="G$1" pin="CS"/>
+<pinref part="U4" gate="G$1" pin="CS"/>
 </segment>
 <segment>
@@
 <net name="RESET_3V3" class="0">
 <segment>
-<pinref part="R6" gate="G$1" pin="2"/>
+<pinref part="R1" gate="G$1" pin="2"/>
 <wire x1="96.52" y1="114.3" x2="104.14" y2="114.3" width="0.1524" layer="91"/>
 <wire x1="104.14" y1="114.3" x2="114.3" y2="114.3" width="0.1524" layer="91"/>
@@
 <wire x1="104.14" y1="106.68" x2="76.2" y2="106.68" width="0.1524" layer="91"/>
 <label x="76.2" y="106.68" size="1.778" layer="95"/>
-<pinref part="U1" gate="G$1" pin="RESET"/>
+<pinref part="U4" gate="G$1" pin="RESET"/>
 </segment>
 <segment>
@@
 <pinref part="R2" gate="G$1" pin="1"/>
 <wire x1="170.18" y1="119.38" x2="172.72" y2="119.38" width="0.1524" layer="91"/>
-<pinref part="U1" gate="G$1" pin="IRQ"/>
-</segment>
-</net>
+<pinref part="U4" gate="G$1" pin="IRQ"/>
+</segment>
+</net>
